File: Kicad/ZX81_32KB_SMD/ZX81_32KB_SMD.kicad_sch (KiCad schematic)
At the start: 4 parts, among them IC1 CY62256NLL-55SNXI, J1 Conn_01x14_Pin, J2 Conn_01x14_Pin, J3 Conn_01x04_Pin

Commit message: Update ZX81_32KB_SMD.kicad_sch
Connections:
- net GND: now also IC1.22 (~{OE})
- net +5V: now reaches J2.10 (Pin_10)
- net +5V: now also IC1.28 (VCC)
- net ~{WR}: now reaches J2.13 (Pin_13)
- net ~{WR}: now also IC1.27 (~{WE})
- net ~{RAMCS}: now reaches J2.6 (Pin_6)
- net ~{RAMCS}: now also IC1.20 (~{CE})
Changed lines of the file:
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@@
+    (effects (font (size 1.27 1.27)) (justify right bottom))
+  )
+  (label "~{RAMCS}" (at 154.94 82.55 180) (fields_autoplaced)
     (effects (font (size 1.27 1.27)) (justify right bottom))
   )
@@
     (effects (font (size 1.27 1.27)) (justify right bottom))
   )
+  (label "~{WR}" (at 154.94 64.77 180) (fields_autoplaced)
+    (effects (font (size 1.27 1.27)) (justify right bottom))
+  )
+  (label "+5V" (at 137.16 62.23 0) (fields_autoplaced)
+    (effects (font (size 1.27 1.27)) (justify left bottom))
+  )
   (label "D7" (at 154.94 95.25 180) (fields_autoplaced)
     (effects (font (size 1.27 1.27)) (justify right bottom))
+  )
+  (label "~{RAMCS}" (at 137.16 82.55 0) (fields_autoplaced)
+    (effects (font (size 1.27 1.27)) (justify left bottom))
   )
   (label "A09" (at 109.22 72.39 180) (fields_autoplaced)
@@
     (effects (font (size 1.27 1.27)) (justify left bottom))
   )
+  (label "~{WR}" (at 137.16 64.77 0) (fields_autoplaced)
+    (effects (font (size 1.27 1.27)) (justify left bottom))
+  )
   (label "A03" (at 154.94 77.47 180) (fields_autoplaced)
     (effects (font (size 1.27 1.27)) (justify right bottom))
@@
   (label "A05" (at 154.94 74.93 180) (fields_autoplaced)
     (effects (font (size 1.27 1.27)) (justify right bottom))
+  )
+  (label "GND" (at 137.16 77.47 0) (fields_autoplaced)
+    (effects (font (size 1.27 1.27)) (justify left bottom))
   )
   (label "A09" (at 87.63 64.77 0) (fields_autoplaced)
@@
     (effects (font (size 1.27 1.27)) (justify left bottom))
   )
+  (label "+5V" (at 154.94 72.39 180) (fields_autoplaced)
+    (effects (font (size 1.27 1.27)) (justify right bottom))
+  )
   (label "A07" (at 87.63 69.85 0) (fields_autoplaced)

Commit message: Update
Parts:
- IC1: footprint SOIC127P1194X279-28N -> CluelessEngineer:DIP1587W140P254L3632H381Q28N; symbol CY62256NLL-55SNXI:CY62256NLL-55SNXI -> AS6C62256-55PCN:AS6C62256-55PCN; Height 2.794 -> 3.81; Manufacturer_Part_Number CY62256NLL-55SNXI -> AS6C62256-55PCN; Mouser Part Number 913-CY62256NLL55SNXI -> 913-AS6C62256-55PCN; Mouser Price/Stock https://www.mouser.co.uk/ProductDetail/Alliance-Memory/CY62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 -> https://www.mouser.co.uk/ProductDetail/Alliance-Memory/AS6C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
- J1, J2: footprint (none) -> Connector_PinHeader_2.54mm:PinHeader_1x14_P2.54mm_Vertical
- J3: footprint (none) -> Connector_PinHeader_2.54mm:PinHeader_1x04_P2.54mm_Horizontal
Connections:
- net +5V: now also J2.12 (Pin_12); no longer J2.10 (Pin_10)
- net A00: now also IC1.10 (A0), J1.10 (Pin_10); no longer IC1.21 (A0), J1.8 (Pin_8)
- net A01: now also IC1.9 (A1), J1.3 (Pin_3); no longer IC1.23 (A1), J1.1 (Pin_1)
- net A02: now also IC1.8 (A2), J1.9 (Pin_9); no longer IC1.24 (A2), J1.7 (Pin_7)
- net A03: now also IC1.7 (A3), J2.10 (Pin_10); no longer IC1.25 (A3), J2.8 (Pin_8)
- net A04: now also IC1.6 (A4), J1.8 (Pin_8); no longer IC1.26 (A4), J1.6 (Pin_6)
- net A05: now also IC1.5 (A5), J2.11 (Pin_11); no longer IC1.1 (A5), J2.9 (Pin_9)
- net A06: now also IC1.4 (A6), J1.7 (Pin_7); no longer IC1.2 (A6), J1.5 (Pin_5)
- net A07: now also J1.6 (Pin_6); no longer J1.4 (Pin_4)
- net A08: now also IC1.25 (A8), J1.5 (Pin_5); no longer IC1.4 (A8), J1.3 (Pin_3)
- net A09: now also IC1.24 (A9), J1.4 (Pin_4); no longer IC1.5 (A9), J1.2 (Pin_2)
- net A10: now also IC1.21 (A10), J2.7 (Pin_7); no longer IC1.6 (A10), J2.14 (Pin_14)
- net A11: now also IC1.23 (A11); no longer IC1.7 (A11)
- net A12: now also IC1.2 (A12); no longer IC1.8 (A12)
- net A13: now also IC1.26 (A13); no longer IC1.9 (A13)
- net A14: now also IC1.1 (A14); no longer IC1.10 (A14)
- net D0: now also J1.11 (Pin_11); no longer J1.9 (Pin_9)
- net D1: now also J1.12 (Pin_12); no longer J1.10 (Pin_10)
- net D2: now also J2.2 (Pin_2); no longer J1.14 (Pin_14)
- net D3: now also J2.4 (Pin_4); no longer J2.2 (Pin_2)
- net D4: now also J2.5 (Pin_5); no longer J2.3 (Pin_3)
- net D5: now also J1.13 (Pin_13); no longer J1.11 (Pin_11)
- net D6: now also J2.1 (Pin_1); no longer J1.13 (Pin_13)
- net D7: now also J2.3 (Pin_3); no longer J2.1 (Pin_1)
- net GND: now also J1.14 (Pin_14); no longer J1.12 (Pin_12)
- net ~{RAMCS}: now also J2.8 (Pin_8)
- net ~{WR}: now also J2.9 (Pin_9); no longer J2.13 (Pin_13)
- no-connect marks 0 -> 4
Other:
- moved on the sheet: IC1
