File: Kicad/ZX81_32KB/ZX81_32KB.kicad_sch (KiCad schematic)
At the start: 4 parts, among them IC1 CY62256NLL-55SNXI, J1 Conn_01x14_Pin, J2 Conn_01x14_Pin, J3 Conn_01x04_Pin

Commit message: Initial version
Other:
- company: (none) -> Brett Hallen
- title: (none) -> ZX81/TS1000 32KB RAM Board
Changed lines of the file:
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@@
 (kicad_sch (version 20230121) (generator eeschema)
   (paper "A4")
+  (title_block
+    (title "ZX81/TS1000 32KB RAM Board")
+    (date "2023-09-10")
+    (rev "INITIAL")
+    (company "Brett Hallen")
+    (comment 1 "youtube.com/@brfff")
+  )
   (no_connect (at 154.94 64.77))
   (no_connect (at 87.63 62.23))
@@
     (pin "9")
     (instances
-      (project "ZX81_32KB_SMD"
+      (project "ZX81_32KB"
         (path "/86e9cda0-559d-4875-9ba4-21806bf6f52d"
           (reference "J2") (unit 1)
@@
     (pin "9")
     (instances
-      (project "ZX81_32KB_SMD"
+      (project "ZX81_32KB"
         (path "/86e9cda0-559d-4875-9ba4-21806bf6f52d"
           (reference "J1") (unit 1)
@@
     (pin "9")
     (instances
-      (project "ZX81_32KB_SMD"
+      (project "ZX81_32KB"
         (path "/86e9cda0-559d-4875-9ba4-21806bf6f52d"
           (reference "IC1") (unit 1)
@@
     (pin "4")
     (instances
-      (project "ZX81_32KB_SMD"
+      (project "ZX81_32KB"
         (path "/86e9cda0-559d-4875-9ba4-21806bf6f52d"
           (reference "J3") (unit 1)
