File: Kicad/ZX81_32KB.kicad_sch (KiCad schematic)
At the start: 4 parts, among them IC1 CY62256NLL-55SNXI, J1 Conn_01x14_Pin, J2 Conn_01x14_Pin, J3 Conn_01x04_Pin

Commit message: Refinements
Parts:
- removed J1, J2: Conn_01x14_Pin, Connector_PinHeader_2.54mm:PinHeader_1x14_P2.54mm_Vertical, symbol Connector:Conn_01x14_Pin
- added J4: 828-AG11D-LF, CluelessEngineer:828AG11DLF, symbol 828-AG11D-LF:828-AG11D-LF
Connections:
- net +5V: now also J4.26
- net A00: now also J4.10
- net A01: now also J4.3
- net A02: now also J4.9
- net A03: now also J4.24
- net A04: now also J4.8
- net A05: now also J4.25
- net A06: now also J4.7
- net A07: now also J4.6
- net A08: now also J4.5
- net A09: now also J4.4
- net A10: now also J4.21
- net D0: now also J4.11
- net D1: now also J4.12
- net D2: now also J4.16
- net D3: now also J4.18
- net D4: now also J4.19
- net D5: now also J4.13
- net D6: now also J4.15
- net D7: now also J4.17
- net GND: now also J4.14; no longer IC1.22 (OE#)
- net ~{RAMCS}: now also IC1.22 (OE#), J4.20, J4.22
- net ~{WR}: now also J4.23
