File: Centronics/Kicad/ZX81_Centronics.kicad_pcb (KiCad board)
At the start: 2 copper layers, 68.8 x 91.4 mm, 19 parts, among them J1 CENTRONICS, Q1 BC558, SW1 SW_Push, U1 74LS27, U2 74LS32, U3 74LS30, U4 8255

Commit message: Updated schematic plot
Connections:
- BUS1 pad GND: (no net) -> GND
Changed lines of the file:
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@@
   )
   (footprint "Capacitor_THT:CP_Radial_D5.0mm_P2.50mm" (layer "F.Cu")
-    (at 145.477113 99.314 180)
+    (at 145.4771 99.314 180)
     (descr "CP, Radial series, Radial, pin pitch=2.50mm, , diameter=5mm, Electrolytic Capacitor")
     (tags "CP Radial series Radial pin pitch 2.50mm  diameter 5mm Electrolytic Capacitor")
@@
     (pad "23B" connect rect (at 20.955 -7.747) (size 1.778 7.62) (layers "B.Cu" "B.Mask")
       (net 31 "/~{ROMCS}") (pinfunction "~{ROM_CS}") (pintype "output"))
-    (pad "GND" connect rect (at -25.9715 -5.9055) (size 2.99974 4.0005) (layers "B.Cu" "B.Mask"))
+    (pad "GND" connect rect (at -25.9715 -5.9055) (size 2.99974 4.0005) (layers "B.Cu" "B.Mask")
+      (net 14 "GND"))
   )
   (gr_line (start 163.83 121.158) (end 152.908 121.158)

Commit message: Generated Gerber files
Parts:
- removed BUS2: PASSTHROUGH, CluelessEngineer:ZX81_EDGE
- moved J1 8.89 mm to (157.2, 70.4)
Connections:
- BUS1 pad GND: GND -> (no net)
Routing:
- net VCC: track 0.00 -> 177.9 mm, vias 0 -> 1
- net /ZX_D0: track 0.00 -> 71.6 mm, vias 0 -> 1
- net /ZX_A0: track 0.00 -> 68.9 mm, vias 0 -> 1
- net /4A: track 0.00 -> 68.1 mm
- net /ZX_A1: track 0.00 -> 67.9 mm, vias 0 -> 1
- net /ZX_D1: track 0.00 -> 67.3 mm, vias 0 -> 1
- net Net-(Q1-B): track 0.00 -> 64.7 mm
- net /1B: track 0.00 -> 63.8 mm
- net /ZX_A5: track 0.00 -> 62.9 mm, vias 0 -> 3
- net /2A: track 0.00 -> 62.3 mm
- net /1A: track 0.00 -> 61.2 mm
- net /ZX_D2: track 0.00 -> 59.0 mm, vias 0 -> 1
- net /ZX_D7: track 0.00 -> 58.6 mm
- net /3B: track 0.00 -> 57.7 mm
- net /2B: track 0.00 -> 57.5 mm
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Other:
- board size 68.8 x 91.4 mm -> 68.8 x 82.5 mm
