File: Centronics/Kicad/ZX81_Centronics.kicad_sch (KiCad schematic)
At the start: 19 parts, among them J1 CENTRONICS, Q1 BC558, SW1 SW_Push, U1 74LS27, U2 74LS32, U3 74LS30, U4 8255

Commit message: Updated schematic plot
Parts:
- C6: footprint (none) -> Capacitor_THT:C_Disc_D4.3mm_W1.9mm_P5.00mm
- SW1: footprint Button_Switch_THT:KSA_Tactile_SPST -> Button_Switch_THT:SW_PUSH_6mm_H4.3mm
Changed lines of the file:
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@@
       (effects (font (size 1.27 1.27)) (justify left))
     )
-    (property "Footprint" "" (at 229.5652 242.57 0)
+    (property "Footprint" "Capacitor_THT:C_Disc_D4.3mm_W1.9mm_P5.00mm" (at 229.5652 242.57 0)
       (effects (font (size 1.27 1.27)) hide)
     )
@@
       (effects (font (size 1.27 1.27)) (justify left))
     )
-    (property "Footprint" "Button_Switch_THT:KSA_Tactile_SPST" (at 59.69 110.49 0)
-      (effects (font (size 1.27 1.27)) hide)
-    )
+    (property "Footprint" "Button_Switch_THT:SW_PUSH_6mm_H4.3mm" (at 59.69 110.49 0)
+      (effects (font (size 1.27 1.27)) hide)
+    )

Commit message: Generated Gerber files
Parts:
- removed BUS2: PASSTHROUGH, CluelessEngineer:ZX81_EDGE, symbol my_components:CONN_ZX81
